File: imxrt10-schematic.kicad_sch (KiCad schematic)
At the start: 89 parts, among them J10 PROG, J11 USB4105-GF-A, J6 MSD-4-A, J8 USB4105-GF-A, J9 Conn_ST_STDC14, SW5 BOOT, SW6 RST, SW7 BOOT, SW8 BOOT, U13 SHT4x, U14 MIMXRT1052DVL6B, U15 USBLC6-2SC6, U16 MCP9701T-E/TT, U17 W25Q128JVS, U18 TPS3839DBZ, U19 USBLC6-2SC6, U20 APS1604M-3SQRx-SN, U22 TPS2051CDBV, X1 Q13FC1350000400, Y3 40MHz, X252040MMB4SI

Commit message: Cleaning the project
Parts:
- added J1: Conn_02x20_Odd_Even, Connector_PinHeader_2.54mm:PinHeader_2x20_P2.54mm_Vertical, symbol Connector_Generic:Conn_02x20_Odd_Even
Connections:
- net GND: now also J1.14 (Pin_14), J1.20 (Pin_20), J1.25 (Pin_25), J1.30 (Pin_30), J1.34 (Pin_34), J1.39 (Pin_39), J1.6 (Pin_6), J1.9 (Pin_9)
- new net: J1.1 (Pin_1), J1.17 (Pin_17)
- new net: J1.2 (Pin_2), J1.4 (Pin_4)

Commit message: Update the source code
Parts:
- removed C45, C68, C92, C98: 100n, Capacitor_SMD:C_0603_1608Metric, symbol Device:C_Small
- removed D10: LED, Yellow, LED_SMD:LED_0603_1608Metric, symbol Device:LED
- removed D8: LED, RED, LED_SMD:LED_0603_1608Metric, symbol Device:LED
- removed D9: LED, White, LED_SMD:LED_0603_1608Metric, symbol Device:LED
- removed J6: MSD-4-A, External_Library:CUI_MSD-4-A, symbol External_Library:MSD-4-A
- removed R29, R30, R38: 750R, Resistor_SMD:R_0603_1608Metric, symbol Device:R
- removed R33, R34: 10K, Resistor_SMD:R_0603_1608Metric, symbol Device:R
- removed U13: SHT4x, Sensor_Humidity:Sensirion_DFN-4_1.5x1.5mm_P0.8mm_SHT4x_NoCentralPad, symbol Sensor_Humidity:SHT4x
- removed U17: W25Q128JVS, Package_SO:SOIC-8_3.9x4.9mm_P1.27mm, symbol Memory_Flash:W25Q128JVS
- removed U20: APS1604M-3SQRx-SN, Package_SO:SOIC-8_3.9x4.9mm_P1.27mm, symbol Memory_RAM:APS1604M-3SQRx-SN
Connections:
- net SPI4_SCK: now reaches U14.B12 (GPIO_B1_07)
- net SPI4_SDO: now reaches U14.C12 (GPIO_B1_06)
- net SPI4_SDI: now reaches U14.D12 (GPIO_B1_05)
- net SPI4_CS0: now reaches U14.E12 (GPIO_B1_04)
- net SPI3_SDO: now reaches U14.G12 (GPIO_AD_B1_14)
- net SPI3_TRG: now reaches U14.H10 (GPIO_AD_B0_01)
- net SPI3_SDI: now reaches U14.H11 (GPIO_AD_B1_13)
- net SPI3_CS0: now reaches U14.H12 (GPIO_AD_B1_12)
- net SPI3_SCK: now reaches U14.J14 (GPIO_AD_B1_15)
- no-connect marks 13 -> 12
Other:
- note removed: "PSRAM"
- note removed: "SD Card"
- note removed: "SPI Flash"
- note removed: "Status LED"
- moved on the sheet: C53, C69, C93, C94, C95, C96, D11, D7, FB2, L3, R25, R27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

Commit message: Update the source code
Parts:
- D7: now not fitted
Connections:
- no-connect marks 12 -> 14
Other:
- note removed: "/**LPUART1 GPIO Configuration PC0 ------> LPUART1_RX PC1 ------> LPUART1_TX */"
Changed lines of the file:
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@@
 		)
 	)
-	(text "  /**LPUART1 GPIO Configuration\n    PC0     ------> LPUART1_RX\n    PC1     ------> LPUART1_TX\n    */"
-		(exclude_from_sim no)
-		(at 57.658 -14.732 0)
-		(effects
-			(font
-				(size 0.762 0.762)
-			)
-		)
-	)
 	(text "IMXRT1170CEC"
 		(exclude_from_sim no)
@@
 		(at 86.36 271.78)
 	)
+	(no_connect
+		(at 151.13 24.13)
+	)
+	(no_connect
+		(at 151.13 21.59)
+	)
 	(wire
 		(pts
@@
 		(exclude_from_sim no)
 		(in_bom yes)
-		(on_board yes)
-		(dnp no)
+		(on_board no)
+		(dnp yes)
 		(property "Reference" "#PWR0112"
 			(at 363.22 214.63 0)
@@
 		(exclude_from_sim no)
 		(in_bom yes)
-		(on_board yes)
-		(dnp no)
+		(on_board no)
+		(dnp yes)
 		(fields_autoplaced yes)
 		(property "Reference" "D7"
@@
 		(exclude_from_sim no)
 		(in_bom yes)
-		(on_board yes)
+		(on_board no)
 		(dnp yes)
 		(fields_autoplaced yes)
@@
 		(exclude_from_sim no)
 		(in_bom yes)
-		(on_board yes)
-		(dnp no)
+		(on_board no)
+		(dnp yes)
 		(property "Reference" "#PWR0110"
 			(at 355.6 207.01 0)
@@
 		(exclude_from_sim no)
 		(in_bom yes)
-		(on_board yes)
-		(dnp no)
+		(on_board no)
+		(dnp yes)
 		(property "Reference" "#PWR0111"
 			(at 355.6 233.68 0)
