File: imxrt10-schematic.kicad_sch (KiCad schematic)
At the start: 73 parts, among them J10 PROG, J11 USB4105-GF-A, J8 USB4105-GF-A, J9 Conn_ST_STDC14, SW5 BOOT, SW6 RST, SW7 BOOT, SW8 BOOT, U14 MIMXRT1052DVL6B, U15 USBLC6-2SC6, U16 MCP9701T-E/TT, U18 TPS3839DBZ, U19 USBLC6-2SC6, U22 TPS2051CDBV, X1 Q13FC1350000400, Y3 40MHz, X252040MMB4SI

Commit message: update the design
Parts:
- removed C80, C89: 100n, Capacitor_SMD:C_0603_1608Metric, symbol Device:C_Small
- removed D11: LED, RED, LED_SMD:LED_0603_1608Metric, symbol Device:LED
- removed FB1: ~, PCM_JLCPCB:FB_0805, symbol PCM_JLCPCB-Inductors:Ferrite,0805,(2)
- removed J10: PROG, Connector_PinHeader_2.54mm:PinHeader_1x04_P2.54mm_Vertical, symbol Connector_Generic:Conn_01x04
- removed R27: 10K, Resistor_SMD:R_0603_1608Metric, symbol Device:R
- removed R31: 750R, Resistor_SMD:R_0603_1608Metric, symbol Device:R
- removed TH2: Thermistor_NTC 10k, Resistor_SMD:R_0805_2012Metric, symbol Device:Thermistor_NTC
- added BT1: Battery_Cell, Battery:BatteryHolder_Keystone_2998_1x6.8mm, symbol Device:Battery_Cell
- added C13: 100n, Capacitor_SMD:C_0402_1005Metric, symbol Device:C_Small
- added D8: LED, RED, LED_SMD:LED_0603_1608Metric, symbol Device:LED
- added D9: LED, White, LED_SMD:LED_0603_1608Metric, symbol Device:LED
- added FB3: ~, PCM_JLCPCB:FB_0603, symbol PCM_JLCPCB-Inductors:Ferrite,0603
- added R11, R16: 750R, Resistor_SMD:R_0603_1608Metric, symbol Device:R
- C101, C103, C104, C53, C54, C55, C57, C59, C61, C62, C63, C64, C69, C72, C75, C76, C77, C78, C81, C82, C83, C84, C85, C86, C87, C88, C90, C91, C97: footprint Capacitor_SMD:C_0603_1608Metric -> Capacitor_SMD:C_0402_1005Metric
- J9: footprint Connector_PinHeader_1.27mm:PinHeader_2x07_P1.27mm_Vertical_SMD -> Connector_PinHeader_1.27mm:PinHeader_2x07_P1.27mm_Vertical; now fitted
- R32, R37: footprint Resistor_SMD:R_0603_1608Metric -> Resistor_SMD:R_0402_1005Metric
Connections:
- net TEM_AN0 is gone; now on net ADC_IN0: U16.2 (Vout)
- net +3.3V: now also C13.1, FB3.2
- net GND: now also BT1.2 (-), C13.2, D8.1 (K), D9.1 (K)
- net VBAT: now also BT1.1 (+)
- net at C73.1, C75.1, U14.N14 (VDDA_ADC_3P3): now also FB3.1
- net MPU_INT: now reaches U14.A12 (GPIO_B1_08)
- net SPI4_TRG: now reaches U14.B14 (GPIO_B1_15)
- net UART3_TX: now reaches U14.B9 (GPIO_B0_08)
- net UART3_RX: now reaches U14.C9 (GPIO_B0_09)
- net GPIO_B1_13_06: now reaches U14.D14 (GPIO_B1_13)
- net CAN_RX: now reaches U14.D8 (GPIO_B0_03)
- net CAN_TX: now reaches U14.E8 (GPIO_B0_02)
- net ADC_IN13: now reaches U14.H13 (GPIO_AD_B1_08)
- net ADC_IN0: now reaches U14.J13 (GPIO_AD_B1_11)
- net ADC_IN10: now reaches U14.K12 (GPIO_AD_B1_05)
- net ADC_IN9: now reaches U14.L12 (GPIO_AD_B1_04)
- net ADC_IN15: now reaches U14.L13 (GPIO_AD_B1_10)
- net ADC_IN14: now reaches U14.M13 (GPIO_AD_B1_09)
- net LED1: now reaches U14.M14 (GPIO_AD_B0_00)
- net LED1: now also R11.2
- net SPI1_SCK: now reaches U14.A2 (GPIO_EMC_27)
- net UART4_CTS: now reaches U14.A4 (GPIO_EMC_17)
- net UART3_RTS: now reaches U14.A5 (GPIO_EMC_16)
- net GPIO_EMC_13: now reaches U14.A6 (GPIO_EMC_13)
- net UART3_CTS: now reaches U14.B1 (GPIO_EMC_15)
- net UART4_RTS: now reaches U14.B2 (GPIO_EMC_18)
- net GPIO_EMC_26: now reaches U14.B3 (GPIO_EMC_26)
- net GPIO_EMC_33: now reaches U14.C4 (GPIO_EMC_33)
- net SPI1_CS0: now reaches U14.C6 (GPIO_EMC_30)
- net SPI1_SDO: now reaches U14.D1 (GPIO_EMC_28)
- net UART5_RX: now reaches U14.D3 (GPIO_EMC_24)
- net GPIO_EMC_32: now reaches U14.D5 (GPIO_EMC_32)
- net GPIO_EMC_38: now reaches U14.D6 (GPIO_EMC_38)
- net SPI1_SDI: now reaches U14.E1 (GPIO_EMC_29)
- net SPI2_SCK: now reaches U14.E3 (GPIO_EMC_00)
- net SPI2_CS0: now reaches U14.F3 (GPIO_EMC_01)
- net SPI2_SDO: now reaches U14.F4 (GPIO_EMC_02)
- net UART5_TX: now reaches U14.G2 (GPIO_EMC_23)
- net SPI2_SDI: now reaches U14.G4 (GPIO_EMC_03)
- net GPIO_EMC_07: now reaches U14.H4 (GPIO_EMC_07)
- new net: D9.2 (A), R16.1
- new net: D8.2 (A), R11.1
- new net LED2: R16.2
Other:
- note added: "Status LED"
- moved on the sheet: R37

Commit message: Update the pcb routing
Connections:
- net GPIO_B1_12: now reaches U14.D13 (GPIO_B1_12)
Changed lines of the file:
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@@
 	(wire
 		(pts
+			(xy 210.82 113.03) (xy 209.55 113.03)
+		)
+		(stroke
+			(width 0)
+			(type default)
+		)
+	)
+	(wire
+		(pts
 			(xy 55.88 252.73) (xy 45.72 252.73)
 		)
@@
 		)
 	)
+	(hierarchical_label "GPIO_B1_12"
+		(shape input)
+		(at 210.82 113.03 0)
+		(effects
+			(font
+				(size 1.27 1.27)
+			)
+			(justify left)
+		)
+	)
