File: esp32c3.kicad_sch (KiCad schematic)
At the start: 27 parts, among them J5 USB4105-GF-A, SW3 BOOT, SW4 BOOT, U6 ESP32-C3FH4, Y2 40MHz, X252040MMB4SI

Commit message: Update the source code
Parts:
- removed J5: USB4105-GF-A, External_Library:GCT_USB4105-GF-A, symbol External_Library:USB4105-GF-A
- removed R11: 10K, Resistor_SMD:R_0603_1608Metric, symbol Device:R
- removed R15, R16: 22R, Resistor_SMD:R_0402_1005Metric, symbol Device:R
- C22, C23, C24, C25, C26, C27, C29: footprint Capacitor_SMD:C_0603_1608Metric -> Capacitor_SMD:C_0402_1005Metric
- R12: footprint Resistor_SMD:R_0603_1608Metric -> Resistor_SMD:R_0402_1005Metric
Connections:
- net ESP_STATUS_LED: no longer U6.8 (GPIO3)
- net RST: now reaches C24.1, R8.2, SW3.1, U6.7 (CHIP_EN)
- net IO5: now reaches U6.10 (MTDI)
- net IO6_SPI_CLK: now reaches U6.12 (MTCK)
- net IO7_SPI_MOSI: now reaches U6.13 (MTDO)
- net IO4_DATA_RDY: now reaches U6.9 (MTMS)
- net ESP_IO10 renamed IO10_CS
- net IO2 renamed IO2_SPI_MISO
- new net IO3_HS: U6.8 (GPIO3)
- no-connect marks 18 -> 10
Other:
- note removed: "ESP32 USB Prog Interface"
- note removed: "The diode will prevent reverse current from the board to the connected PC portwhen the power is already powered."

Commit message: update the design
Parts:
- removed C25: 100n, Capacitor_SMD:C_0402_1005Metric, symbol Device:C_Small
- added J3, J4: Conn_01x07, Connector_PinSocket_2.54mm:PinSocket_1x07_P2.54mm_Vertical, symbol Connector_Generic:Conn_01x07
- R13, R14, R8: footprint Resistor_SMD:R_0603_1608Metric -> Resistor_SMD:R_0402_1005Metric
Connections:
- net ESP_RX: now also J4.7 (Pin_7)
- net ESP_STATUS_LED: now also U6.4 (XTAL_32K_P)
- net ESP_TX: now also J3.7 (Pin_7)
- net GND: now also J4.2 (Pin_2)
- net IO10_CS: now also J4.4 (Pin_4)
- net IO2_SPI_MISO: now also J3.1 (Pin_1)
- net IO3_HS: now also J3.2 (Pin_2)
- net IO4_DATA_RDY: now also J3.3 (Pin_3)
- net IO5: now also J3.4 (Pin_4)
- net IO6_SPI_CLK: now also J3.5 (Pin_5)
- net IO7_SPI_MOSI: now also J3.6 (Pin_6)
- net IO8: now also J4.6 (Pin_6)
- net IO9: now also J4.5 (Pin_5)
- no-connect marks 10 -> 9
Other:
- moved on the sheet: C28, C29
