File: power-supply.kicad_sch (KiCad schematic)
At the start: 11 parts, among them U7 AMS1117-3.3, U8 AP63203WU

Commit message: Update the pcb routing
Parts:
- removed JP2: JUMP, External_Library:power-jumper-3, symbol Jumper:Jumper_3_Open
Connections:
- net VIN: now also C32.1, C34.1, C35.1, U7.3 (VI), U8.2 (EN), U8.3 (IN)
Changed lines of the file:
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@@
+	)
+	(junction
+		(at 68.58 57.15)
+		(diameter 0)
+		(color 0 0 0 0)
 	)
 	(junction
@@
 	(wire
 		(pts
-			(xy 68.58 63.5) (xy 68.58 69.85)
+			(xy 68.58 49.53) (xy 68.58 57.15)
 		)
 		(stroke
@@
 	(wire
 		(pts
+			(xy 68.58 57.15) (xy 68.58 69.85)
+		)
+		(stroke
+			(width 0)
+			(type default)
+		)
+	)
+	(wire
+		(pts
 			(xy 87.63 69.85) (xy 93.98 69.85)
 		)
@@
 	(wire
 		(pts
-			(xy 58.42 57.15) (xy 64.77 57.15)
+			(xy 58.42 57.15) (xy 68.58 57.15)
 		)
 		(stroke
@@
 		(pts
 			(xy 105.41 55.88) (xy 107.95 55.88)
-		)
-		(stroke
-			(width 0)
-			(type default)
-		)
-	)
-	(wire
-		(pts
-			(xy 68.58 49.53) (xy 68.58 50.8)
 		)
 		(stroke
@@
 					(unit 1)
 				)
-			)
-		)
-	)
-	(symbol
-		(lib_id "Jumper:Jumper_3_Open")
-		(at 68.58 57.15 270)
-		(unit 1)
-		(exclude_from_sim yes)
-		(in_bom no)
-		(on_board yes)
-		(dnp yes)
-		(fields_autoplaced yes)
-		(property "Reference" "JP2"
-			(at 71.12 55.8799 90)
-			(effects
-				(font
-					(size 1.27 1.27)
-				)
-				(justify left)
-			)
-		)
-		(property "Value" "JUMP"
-			(at 71.12 58.4199 90)
-			(effects
-				(font
-					(size 1.27 1.27)
-				)
-				(justify left)
-			)
-		)
-		(property "Footprint" "External_Library:power-jumper-3"
-			(at 68.58 57.15 0)
-			(effects
-				(font
-					(size 1.27 1.27)
-				)
-				(hide yes)
-			)
-		)
-		(property "Datasheet" "~"
-			(at 68.58 57.15 0)
-			(effects
-				(font
-					(size 1.27 1.27)
-				)
-				(hide yes)
-			)
-		)
-		(property "Description" "Jumper, 3-pole, both open"
-			(at 68.58 57.15 0)
-			(effects
-				(font
-					(size 1.27 1.27)
-				)
-				(hide yes)
-			)
-		)
-		(property "LCSC Part" "~"
-			(at 68.58 57.15 0)
-			(effects
-				(font
-					(size 1.27 1.27)
-				)
-				(hide yes)
-			)
-		)
-		(pin "1"
-		)
-		(pin "3"
-		)
-		(pin "2"
-		)
-		(instances
-			(project "imxrt10-mcu-board-design"
-				(path "/72ac21c7-a543-4794-a410-99cf6f99d934/24935dec-f667-4a7b-81ef-9ba642ab8f82"
-					(reference "JP2")
-					(unit 1)
-				)
