File: imxrt10-mcu-board-design.kicad_pcb (KiCad board)
At the start: 4 copper layers, 100 x 59.8 mm, 171 parts, among them J10 PROG, J11 USB4105-GF-A, J4 PROG, J5 USB4105-GF-A, J6 MSD-4-A, J7 PROG, J8 USB4105-GF-A, J9 Conn_ST_STDC14, SW1 BOOT, SW3 BOOT, SW4 BOOT, SW5 BOOT, SW6 RST, SW7 BOOT, SW8 BOOT, U10 ADXL343, U11 WIZFI360-PA, U13 SHT4x, U14 MIMXRT1052DVL6B, U15 USBLC6-2SC6, U16 MCP9701T-E/TT, U17 W25Q128JVS, U18 TPS3839DBZ, U19 USBLC6-2SC6, U20 APS1604M-3SQRx-SN, U22 TPS2051CDBV, U4 SHT4x, U5 MCP9701T-E/TT, U6 ESP32-C3FH4, U7 AMS1117-3.3, U8 AP63203WU, X1 Q13FC1350000400, Y2 40MHz, X252040MMB4SI, Y3 40MHz, X252040MMB4SI

Commit message: Cleaning the project
Parts:
- removed C2, C20: 100n, Capacitor_SMD:C_0603_1608Metric
- removed J4, J7: PROG, Connector_PinHeader_2.54mm:PinHeader_1x04_P2.54mm_Vertical
- removed R1: 10K, Resistor_SMD:R_0603_1608Metric
- removed SW1: BOOT, Button_Switch_SMD:SW_SPST_TL3342
- removed U4: SHT4x, Sensor_Humidity:Sensirion_DFN-4_1.5x1.5mm_P0.8mm_SHT4x_NoCentralPad
- added C47: 100n, Capacitor_SMD:C_0603_1608Metric, F.Cu at (28.2, 0.76)
- added C49: 10uF, Capacitor_SMD:C_0603_1608Metric, F.Cu at (28.2, 3.27)
- added J1: Conn_02x20_Odd_Even, Connector_PinHeader_2.54mm:PinHeader_2x20_P2.54mm_Vertical, F.Cu at (150.8, 118.2)
- added U1: ESP32-C3-DevKitM-1, RF_Module:ESP32-C3-DevKitM-1, F.Cu at (1.43, 7.38)
- SW3, SW4: footprint Button_Switch_SMD:SW_SPST_TL3342 -> Button_Switch_SMD:SW_SPST_B3U-1000P-B
- moved G*** 36.9 mm to (186.8, 55.5)
- moved TH1 14.0 mm to (171.0, 74.0)
- moved R3 14.0 mm to (170.8, 75.8)
- moved C21 14.0 mm to (175.8, 70.9)
- moved D1 14.0 mm to (171.5, 69.7)
- moved C40 12.2 mm to (169.7, 92.6)
- moved C43 12.2 mm to (169.7, 91.0)
- moved AE1 11.6 mm to (205.5, 100.2)
- moved C28 11.6 mm to (186.9, 106.0)
- moved D6 11.6 mm to (190.1, 107.4)
- moved R12 11.6 mm to (190.5, 97.0)
- moved R16 11.6 mm to (193.0, 107.9)
- moved R21 11.6 mm to (176.3, 95.3)
- moved R5 11.6 mm to (171.6, 104.0)
- moved R8 11.6 mm to (188.1, 98.7)
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Connections:
- U14 pad A11: unconnected-(U14D-GPIO_B1_00-PadA11) -> /imxrt10-schematic/UART4_RX
- U14 pad B11: unconnected-(U14D-GPIO_B1_01-PadB11) -> /imxrt10-schematic/UART4_TX
- U14 pad B8: unconnected-(U14D-GPIO_B0_05-PadB8) -> /imxrt10-schematic/I2C2_SDA
- U14 pad C8: unconnected-(U14D-GPIO_B0_04-PadC8) -> /imxrt10-schematic/I2C2_SCL
- U14 pad G11: unconnected-(U14E-GPIO_AD_B0_03-PadG11) -> /imxrt10-schematic/UART6_RX
- U14 pad H14: unconnected-(U14E-GPIO_AD_B0_14-PadH14) -> /imxrt10-schematic/USB_HOST_PWR_OC
- U14 pad J11: unconnected-(U14E-GPIO_AD_B1_00-PadJ11) -> /imxrt10-schematic/I2C1_SCL
- U14 pad J12: unconnected-(U14E-GPIO_AD_B1_06-PadJ12) -> /imxrt10-schematic/I2C3_SDA
- U14 pad K10: unconnected-(U14E-GPIO_AD_B1_07-PadK10) -> /imxrt10-schematic/I2C3_SCL
- U14 pad K11: unconnected-(U14E-GPIO_AD_B1_01-PadK11) -> /imxrt10-schematic/I2C1_SDA
- U14 pad K14: unconnected-(U14E-GPIO_AD_B0_12-PadK14) -> /imxrt10-schematic/I2C4_SCL
- U14 pad L10: unconnected-(U14E-GPIO_AD_B0_15-PadL10) -> /imxrt10-schematic/USB_HOST_PWR_EN
- U14 pad L11: unconnected-(U14E-GPIO_AD_B1_02-PadL11) -> /imxrt10-schematic/UART2_TX
- U14 pad L14: unconnected-(U14E-GPIO_AD_B0_13-PadL14) -> /imxrt10-schematic/I2C4_SDA
- U14 pad M11: unconnected-(U14E-GPIO_AD_B0_02-PadM11) -> /imxrt10-schematic/UART6_TX
- U14 pad M12: unconnected-(U14E-GPIO_AD_B1_03-PadM12) -> /imxrt10-schematic/UART2_RX
Routing:
- net GND: track 40.0 -> 38.6 mm, vias 31 -> 30

Commit message: Update the source code
Parts:
- removed J5: USB4105-GF-A, External_Library:GCT_USB4105-GF-A
- removed R11: 10K, Resistor_SMD:R_0603_1608Metric
- removed R15, R16: 22R, Resistor_SMD:R_0402_1005Metric
- added R1: 10K, Resistor_SMD:R_0603_1608Metric, F.Cu at (155.6, 89.4)
- added R2: 10K, Resistor_SMD:R_0603_1608Metric, F.Cu at (155.6, 91.9)
- C22, C23, C24, C25, C26, C27, C29: footprint Capacitor_SMD:C_0603_1608Metric -> Capacitor_SMD:C_0402_1005Metric
- R12: footprint Resistor_SMD:R_0603_1608Metric -> Resistor_SMD:R_0402_1005Metric
- moved R38 84.5 mm to (159.6, 89.4)
- moved C45 79.8 mm to (155.6, 79.4)
- moved C98 78.7 mm to (155.6, 86.9)
- moved R33 77.7 mm to (159.6, 84.4)
- moved R34 77.7 mm to (159.6, 86.9)
- moved C68 55.7 mm to (155.6, 81.9)
- moved R29 51.1 mm to (159.6, 79.4)
- moved R30 51.1 mm to (159.6, 81.9)
- moved C92 48.6 mm to (155.6, 84.4)
- moved U13 39.2 mm to (163.7, 87.4)
- moved D10 31.2 mm to (163.7, 84.6)
- moved D8 31.2 mm to (163.7, 79.4)
- moved D9 31.2 mm to (163.7, 82.0)
- moved U17 25.9 mm to (157.8, 96.5), turned to 0 degrees
- moved U20 15.8 mm to (157.8, 103.1)
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Connections:
- net Net-(U6-CHIP_EN) renamed /esp32_wifi_section/RST
- R10 pad 1: /USART1_RX -> /esp32_wifi_section/ESP_TX
- R29 pad 2: /imxrt10-schematic/LED2 -> /LED2
- R30 pad 2: /imxrt10-schematic/LED3 -> /LED3
- R38 pad 2: /imxrt10-schematic/LED1 -> /LED1
- R9 pad 1: /USART1_TX -> /esp32_wifi_section/ESP_RX
- U13 pad 1: /imxrt10-schematic/I2C1_SDA -> /I2C1_SDA
- U13 pad 2: /imxrt10-schematic/I2C1_SCL -> /I2C1_SCL
- U14 pad B12: unconnected-(U14D-GPIO_B1_07-PadB12) -> /imxrt10-schematic/SPI4_SCK
- U14 pad C12: unconnected-(U14D-GPIO_B1_06-PadC12) -> /imxrt10-schematic/SPI4_SDO
- U14 pad D12: unconnected-(U14D-GPIO_B1_05-PadD12) -> /imxrt10-schematic/SPI4_SDI
- U14 pad E12: unconnected-(U14D-GPIO_B1_04-PadE12) -> /imxrt10-schematic/SPI4_CS0
- U14 pad G11: /imxrt10-schematic/UART6_RX -> /esp32_wifi_section/ESP_TX
- U14 pad G12: unconnected-(U14E-GPIO_AD_B1_14-PadG12) -> /esp32_wifi_section/IO7_SPI_MOSI
- U14 pad H10: unconnected-(U14E-GPIO_AD_B0_01-PadH10) -> /esp32_wifi_section/IO4_DATA_RDY
- U14 pad H11: unconnected-(U14E-GPIO_AD_B1_13-PadH11) -> /esp32_wifi_section/IO2_SPI_MISO
- U14 pad H12: unconnected-(U14E-GPIO_AD_B1_12-PadH12) -> /esp32_wifi_section/IO10_CS
- U14 pad J11: /imxrt10-schematic/I2C1_SCL -> /I2C1_SCL
- U14 pad J14: unconnected-(U14E-GPIO_AD_B1_15-PadJ14) -> /esp32_wifi_section/IO6_SPI_CLK
- U14 pad K11: /imxrt10-schematic/I2C1_SDA -> /I2C1_SDA
- U14 pad M11: /imxrt10-schematic/UART6_TX -> /esp32_wifi_section/ESP_RX
- U6 pad 10: unconnected-(U6-MTDI-Pad10) -> /esp32_wifi_section/IO5
- U6 pad 12: unconnected-(U6-MTCK-Pad12) -> /esp32_wifi_section/IO6_SPI_CLK
- U6 pad 13: unconnected-(U6-MTDO-Pad13) -> /esp32_wifi_section/IO7_SPI_MOSI
- U6 pad 16: /esp32_wifi_section/ESP_IO10 -> /esp32_wifi_section/IO10_CS
- U6 pad 6: /esp32_wifi_section/IO2 -> /esp32_wifi_section/IO2_SPI_MISO
- U6 pad 8: ESP_STATUS_LED -> /esp32_wifi_section/IO3_HS
- U6 pad 9: unconnected-(U6-MTMS-Pad9) -> /esp32_wifi_section/IO4_DATA_RDY
Routing:
- net +3.3V: track 41.5 -> 5.79 mm, vias 9 -> 2
- net Net-(U11-TXD1/IIC_SDA): track 34.4 -> 0.00 mm
- net Net-(U11-RXD1/IIC_SCL): track 31.9 -> 0.00 mm
- net /esp32_wifi_section/RST: track 29.9 -> 0.00 mm, vias 3 -> 0
- net Net-(U6-U0RXD): track 28.6 -> 0.00 mm, vias 2 -> 0
- net Net-(U6-U0TXD): track 27.2 -> 0.00 mm, vias 2 -> 0
- net Net-(U11-PB10/RTSI): track 23.1 -> 0.00 mm
- net GND: track 38.6 -> 16.4 mm, vias 30 -> 20
- net /esp32_wifi_section/_USB_D+: track 22.2 -> 0.00 mm, vias 1 -> 0
- net /esp32_wifi_section/_USB_D-: track 21.7 -> 0.00 mm, vias 1 -> 0
- net Net-(D6-A): track 18.6 -> 0.00 mm, vias 2 -> 0
- net Net-(U11-PB9/CTS1): track 15.7 -> 0.00 mm
- net /esp32_wifi_section/IO9: track 11.7 -> 0.00 mm
- net /USART3_RX: track 9.61 -> 0.00 mm
- net /esp32_wifi_section/XTAL_P: track 8.41 -> 0.00 mm
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
Commit message: Update the source code
Parts:
- removed C21, C69: 100n, Capacitor_SMD:C_0603_1608Metric
- removed D1, D7: Inolux_IN-PI554FCH, LED_SMD:LED_Inolux_IN-PI554FCH_PLCC4_5.0x5.0mm_P3.2mm
- added C11: 100n, Capacitor_SMD:C_0402_1005Metric, F.Cu at (181.0, 70.0)
- added C2: 2.2u, Capacitor_SMD:C_0402_1005Metric, F.Cu at (203.5, 43.1)
- added C20: 22u, Capacitor_SMD:C_0603_1608Metric, F.Cu at (199.7, 33.3)
- added C3: 2.2u, Capacitor_SMD:C_0402_1005Metric, F.Cu at (203.5, 45.1)
- added C56: 10uF, Capacitor_SMD:C_0603_1608Metric, F.Cu at (199.7, 35.8)
- added C58: 2.2u, Capacitor_SMD:C_0402_1005Metric, F.Cu at (203.5, 49.0)
- added C6: 10uF, Capacitor_SMD:C_0603_1608Metric, F.Cu at (195.6, 33.3)
- added C60: 100n, Capacitor_SMD:C_0603_1608Metric, F.Cu at (199.7, 38.3)
- added C67: 100n, Capacitor_SMD:C_0603_1608Metric, F.Cu at (203.7, 33.3)
- added C7: 2.2u, Capacitor_SMD:C_0402_1005Metric, F.Cu at (203.5, 47.0)
- added C70: 100n, Capacitor_SMD:C_0603_1608Metric, F.Cu at (203.7, 35.8)
- added C8: 100n, Capacitor_SMD:C_0603_1608Metric, F.Cu at (195.6, 35.8)
- added C9: 100n, Capacitor_SMD:C_0603_1608Metric, F.Cu at (195.6, 38.3)
- added D16: LED WS2812B, LED_SMD:LED_WS2812B_PLCC4_5.0x5.0mm_P3.2mm, F.Cu at (134.0, 104.2)
- added R15: 10K, Resistor_SMD:R_0402_1005Metric, F.Cu at (178.1, 67.0)
- added R39: 10K, Resistor_SMD:R_0603_1608Metric, F.Cu at (203.7, 38.3)
- added R40: 10K, Resistor_SMD:R_0402_1005Metric, F.Cu at (178.1, 69.0)
- added R49: 10K, Resistor_SMD:R_0603_1608Metric, F.Cu at (203.7, 40.9)
- added U30: STM32F103C8Tx, Package_QFP:LQFP-48_7x7mm_P0.5mm, F.Cu at (169.8, 71.5)
- added U4: SHT4x, Sensor_Humidity:Sensirion_DFN-4_1.5x1.5mm_P0.8mm_SHT4x_NoCentralPad, F.Cu at (181.6, 67.5)
- added U9: W9812G6KH-5, Package_SO:TSOP-II-54_22.2x10.16mm_P0.8mm, F.Cu at (152.3, 105.8)
- moved U5 81.1 mm to (178.6, 32.2), turned to 0 degrees
- moved TH1 13.4 mm to (180.5, 83.5)
- moved R3 13.4 mm to (180.3, 85.3)
- moved U10 12.1 mm to (178.0, 79.5)
Connections:
- U11 pad 10: unconnected-(U11-PB18/SPI_MISO-Pad10) -> /modules-sections/WIZ_SPI_MISO
- U11 pad 12: unconnected-(U11-PB14/SPI_INT-Pad12) -> /modules-sections/WIZ_SPI_INT
- U11 pad 13: unconnected-(U11-PB17_SPI/MOSI-Pad13) -> /modules-sections/WIZ_SPI_MOSI
- U11 pad 14: unconnected-(U11-PB16/SPI_CK-Pad14) -> /modules-sections/WIZ_SPI_SCK
- U11 pad 9: unconnected-(U11-PB15/SPI_CS-Pad9) -> /modules-sections/WIZ_SPI_CS
- U5 pad 2: TEM_AN0 -> /stm32f103-mcu-interface/TH_Sensor

Commit message: update the design
Parts:
- removed C25: 100n, Capacitor_SMD:C_0402_1005Metric
- removed C56: 10uF, Capacitor_SMD:C_0603_1608Metric
- removed C58: 2.2u, Capacitor_SMD:C_0402_1005Metric
- removed C67, C80, C89: 100n, Capacitor_SMD:C_0603_1608Metric
- removed D11, D2: LED, RED, LED_SMD:LED_0603_1608Metric
- removed D3: LED, White, LED_SMD:LED_0603_1608Metric
- removed D4: LED, Yellow, LED_SMD:LED_0603_1608Metric
- removed FB1: ~, PCM_JLCPCB:FB_0805
- removed J10: PROG, Connector_PinHeader_2.54mm:PinHeader_1x04_P2.54mm_Vertical
- removed JP4, JP5: JP, Jumper:SolderJumper-2_P1.3mm_Open_RoundedPad1.0x1.5mm
- removed R30, R31, R38, R4, R5, R6: 750R, Resistor_SMD:R_0603_1608Metric
- removed TH2: Thermistor_NTC 10k, Resistor_SMD:R_0805_2012Metric
- removed U1: ESP32-C3-DevKitM-1, RF_Module:ESP32-C3-DevKitM-1
- removed U9: W9812G6KH-5, Package_SO:TSOP-II-54_22.2x10.16mm_P0.8mm
- added BT1: Battery_Cell, Battery:BatteryHolder_Keystone_2998_1x6.8mm, F.Cu at (131.2, 97.2)
- added C1: 100n, Capacitor_SMD:C_0603_1608Metric, F.Cu at (182.3, 57.5)
- added C10: 470n, Capacitor_SMD:C_0603_1608Metric, F.Cu at (184.9, 60.1)
- added C12: 10u, Capacitor_SMD:C_0805_2012Metric, F.Cu at (182.5, 59.4)
- added C13: 100n, Capacitor_SMD:C_0402_1005Metric, F.Cu at (150.1, 100.8)
- added C4: 470n, Capacitor_SMD:C_0603_1608Metric, F.Cu at (182.4, 67.6)
- added C5: 10u, Capacitor_SMD:C_0805_2012Metric, F.Cu at (182.6, 65.8)
- added D13: SS34, PCM_JLCPCB:D_SMA, F.Cu at (127.3, 109.2)
- added FB3: ~, PCM_JLCPCB:FB_0603, F.Cu at (154.6, 96.8)
- added H1: MountingHole_Pad, MountingHole:MountingHole_2.5mm_Pad, F.Cu at (114.0, 50.0)
- added H2: MountingHole_Pad, MountingHole:MountingHole_2.5mm_Pad, F.Cu at (208.0, 50.0)
- added H3: MountingHole_Pad, MountingHole:MountingHole_2.5mm_Pad, F.Cu at (114.0, 118.0)
- added H4: MountingHole_Pad, MountingHole:MountingHole_2.5mm_Pad, F.Cu at (208.0, 118.0)
- added J2: Conn_ST_STDC14, Connector_PinHeader_1.27mm:PinHeader_2x07_P1.27mm_Vertical, F.Cu at (172.6, 57.3)
- added J3: Conn_01x07, Connector_PinSocket_2.54mm:PinSocket_1x07_P2.54mm_Vertical, F.Cu at (201.5, 77.8)
- added J4: Conn_01x07, Connector_PinSocket_2.54mm:PinSocket_1x07_P2.54mm_Vertical, F.Cu at (201.5, 93.0)
- added Q1: HL3401, PCM_JLCPCB:Q_SOT-23, F.Cu at (154.1, 55.0)
- added Q2: HL3401, PCM_JLCPCB:Q_SOT-23, F.Cu at (168.2, 109.4)
- added Q3: HL3401, PCM_JLCPCB:Q_SOT-23, F.Cu at (186.9, 51.6)
- added Q4: 2N7002K, PCM_JLCPCB:Q_SOT-23, F.Cu at (154.0, 60.5)
- added Q5: 2N7002K, PCM_JLCPCB:Q_SOT-23, F.Cu at (181.9, 51.1)
- added Q6: 2N7002K, PCM_JLCPCB:Q_SOT-23, F.Cu at (162.7, 109.2)
- added Q7: 2N7002K, PCM_JLCPCB:Q_SOT-23, F.Cu at (179.6, 84.2)
- added Q8: HL3401, PCM_JLCPCB:Q_SOT-23, F.Cu at (183.7, 84.2)
- added R11: 750R, Resistor_SMD:R_0603_1608Metric, F.Cu at (140.4, 102.8)
- added R16: 750R, Resistor_SMD:R_0603_1608Metric, F.Cu at (142.9, 102.8)
- added R41: 10K, Resistor_SMD:R_0603_1608Metric, F.Cu at (153.9, 57.7)
- added R45: 10K, Resistor_SMD:R_0603_1608Metric, F.Cu at (165.4, 109.3)
- added R46: 10K, Resistor_SMD:R_0402_1005Metric, F.Cu at (184.4, 51.4)
- added U2: SPX3819M5-L-3-3, Package_TO_SOT_SMD:SOT-23-5, F.Cu at (182.5, 62.5)
- C101, C103, C104, C39, C53, C54, C55, C57, C59, C61, C62, C63, C64, C68, C72, C75, C76, C77, C78, C81, C83, C85, C86, C87, C88, C90, C91, C97: footprint Capacitor_SMD:C_0603_1608Metric -> Capacitor_SMD:C_0402_1005Metric
- C79: moved to B.Cu
- C82, C84: footprint Capacitor_SMD:C_0603_1608Metric -> Capacitor_SMD:C_0402_1005Metric; moved to B.Cu
- J9: footprint Connector_PinHeader_1.27mm:PinHeader_2x07_P1.27mm_Vertical_SMD -> Connector_PinHeader_1.27mm:PinHeader_2x07_P1.27mm_Vertical
- R1, R13, R14, R17, R18, R2, R32, R37, R8: footprint Resistor_SMD:R_0603_1608Metric -> Resistor_SMD:R_0402_1005Metric
- R27: value 10K -> 750R
- R29: value 750R -> 10K; footprint Resistor_SMD:R_0603_1608Metric -> Resistor_SMD:R_0402_1005Metric
- moved C49 172.4 mm to (193.5, 52.5)
- moved C47 169.8 mm to (190.4, 50.8), turned to 180 degrees
- moved SW8 111.5 mm to (114.8, 79.3), turned to 180 degrees
- moved SW7 111.5 mm to (114.8, 72.0), turned to 180 degrees
- moved R26 109.9 mm to (127.5, 87.7)
- moved C102 109.5 mm to (124.2, 67.0), turned to 180 degrees
- moved U18 109.0 mm to (124.8, 84.8)
- moved C55 108.8 mm to (124.4, 82.2), turned to 180 degrees
- moved C103 91.0 mm to (149.3, 86.2), turned to 180 degrees
- moved C57 90.3 mm to (145.2, 86.7), turned to 90 degrees
- moved C97 90.0 mm to (145.2, 88.5), turned to -90 degrees
- moved C104 89.5 mm to (149.3, 85.2), turned to 180 degrees
- moved R37 87.9 mm to (159.8, 94.2), turned to -90 degrees
- moved C53 74.7 mm to (119.8, 95.4), turned to 90 degrees
- moved C64 72.4 mm to (164.4, 88.8)
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Connections:
- net Net-(J1-Pin_1) renamed +3.3V_EXT
- net Net-(JP5-B) renamed +3.3V_WIFI
- C11 pad 1: +3.3V -> +3.3V1
- C2 pad 1: VDD -> +3.3V1
- C20 pad 1: VDD -> +3.3V1
- C3 pad 1: VDD -> +3.3V1
- C39 pad 1: /modules-sections/VDD -> +3.3V1
- C40 pad 1: /modules-sections/VDD -> +3.3V1
- C43 pad 1: /modules-sections/VDD -> +3.3V1
- C45 pad 1: +3.3V -> +3.3V_SD
- C6 pad 1: VDD -> +3.3V1
- C60 pad 1: +3.3V -> +3.3V1
- C7 pad 1: VDD -> +3.3V1
- C8 pad 1: VDD -> +3.3V1
- C9 pad 1: VDD -> +3.3V1
- D16 pad 1: VDD -> +3.3V1
- J1 pad 10: unconnected-(J1-Pin_10-Pad10) -> /EXT_IO15_UART1_TX
- J1 pad 11: unconnected-(J1-Pin_11-Pad11) -> /EXT_IO17_UART1_CTS
- J1 pad 12: unconnected-(J1-Pin_12-Pad12) -> /EXT_IO18
- J1 pad 13: unconnected-(J1-Pin_13-Pad13) -> /EXT_IO27
- J1 pad 15: unconnected-(J1-Pin_15-Pad15) -> /EXT_IO22
- J1 pad 16: unconnected-(J1-Pin_16-Pad16) -> /EXT_IO23_CAN_TX
- J1 pad 18: unconnected-(J1-Pin_18-Pad18) -> /EXT_IO24_CAN_RX
- J1 pad 19: unconnected-(J1-Pin_19-Pad19) -> /EXT_IO10_SPI_MOSI
- J1 pad 21: unconnected-(J1-Pin_21-Pad21) -> /EXT_IO9_SPI_MISO
- J1 pad 22: unconnected-(J1-Pin_22-Pad22) -> /EXT_IO25
- J1 pad 23: unconnected-(J1-Pin_23-Pad23) -> /EXT_IO11_SPI_SCK
- J1 pad 24: unconnected-(J1-Pin_24-Pad24) -> /EXT_IO8_SPI_CS
- J1 pad 26: unconnected-(J1-Pin_26-Pad26) -> /EXT_IO7
- J1 pad 27: unconnected-(J1-Pin_27-Pad27) -> /EXT_IO1_I2C0_SDA
- J1 pad 28: unconnected-(J1-Pin_28-Pad28) -> /EXT_IO0_I2C0_SCL
- J1 pad 29: unconnected-(J1-Pin_29-Pad29) -> /EXT_IO5
- J1 pad 3: unconnected-(J1-Pin_3-Pad3) -> /EXT_IO2_I2C1_SDA
- J1 pad 31: unconnected-(J1-Pin_31-Pad31) -> /EXT_IO6
- J1 pad 32: unconnected-(J1-Pin_32-Pad32) -> /EXT_IO12
- J1 pad 33: unconnected-(J1-Pin_33-Pad33) -> /EXT_IO13_UART2_TX
- J1 pad 35: unconnected-(J1-Pin_35-Pad35) -> /EXT_IO19
- J1 pad 36: unconnected-(J1-Pin_36-Pad36) -> /EXT_IO16_UART1_RTS
- J1 pad 37: unconnected-(J1-Pin_37-Pad37) -> /EXT_IO26_UART2_RX
- J1 pad 38: unconnected-(J1-Pin_38-Pad38) -> /EXT_IO20
- J1 pad 40: unconnected-(J1-Pin_40-Pad40) -> /EXT_IO21
- J1 pad 5: unconnected-(J1-Pin_5-Pad5) -> /EXT_IO3_I2C1_SCL
- J1 pad 7: unconnected-(J1-Pin_7-Pad7) -> /EXT_IO4
- J1 pad 8: unconnected-(J1-Pin_8-Pad8) -> /EXT_IO14_UART1_RX
- J6 pad 4: +3.3V -> +3.3V_SD
- J9 pad 13: /imxrt10-schematic/UART2_RX -> /EXT_IO13_UART2_TX
- J9 pad 14: /imxrt10-schematic/UART2_TX -> /EXT_IO26_UART2_RX
- R1 pad 2: /I2C1_SCL -> /EXT_IO0_I2C0_SCL
- R12 pad 2: ESP_STATUS_LED -> /esp32_wifi_section/ESP_STATUS_LED
- R15 pad 1: +3.3V -> +3.3V1
- R17 pad 1: /modules-sections/VDD -> +3.3V1
- R17 pad 2: /I2C1_SDA -> /imxrt10-schematic/I2C2_SDA
- R18 pad 1: /modules-sections/VDD -> +3.3V1
- R18 pad 2: /I2C1_SCL -> /imxrt10-schematic/I2C2_SCL
- R2 pad 2: /I2C1_SDA -> /EXT_IO1_I2C0_SDA
- R27 pad 1: +3.3V -> Net-(D10-A)
- R27 pad 2: /imxrt10-schematic/NTC_TEMP -> /stm32f103-mcu-interface/LED3
- R29 pad 1: Net-(D9-A) -> +3.3V_SYS
- R29 pad 2: /LED2 -> Net-(Q7-D)
- R3 pad 1: +3.3V -> +3.3V1
- R3 pad 2: /NTC_TEMP -> /stm32f103-mcu-interface/NTC_TEMP
- R39 pad 1: VDD -> +3.3V1
- R40 pad 1: +3.3V -> +3.3V1
- TH1 pad 1: /NTC_TEMP -> /stm32f103-mcu-interface/NTC_TEMP
- U10 pad 1: /modules-sections/VDD -> +3.3V1
- U10 pad 13: /I2C1_SDA -> /imxrt10-schematic/I2C2_SDA
- U10 pad 14: /I2C1_SCL -> /imxrt10-schematic/I2C2_SCL
- U10 pad 6: /modules-sections/VDD -> +3.3V1
- U10 pad 7: /modules-sections/VDD -> +3.3V1
- U13 pad 1: /I2C1_SDA -> /EXT_IO1_I2C0_SDA
- U13 pad 2: /I2C1_SCL -> /EXT_IO0_I2C0_SCL
- U14 pad A11: /imxrt10-schematic/UART4_RX -> /USART3_TX
- U14 pad A2: unconnected-(U14G-GPIO_EMC_27-PadA2) -> /imxrt10-schematic/SPI1_SCK
- U14 pad A4: unconnected-(U14G-GPIO_EMC_17-PadA4) -> /USART3_CTS
- U14 pad A5: unconnected-(U14G-GPIO_EMC_16-PadA5) -> /EXT_IO17_UART1_CTS
- U14 pad A6: unconnected-(U14G-GPIO_EMC_13-PadA6) -> /EXT_IO20
- U14 pad B1: unconnected-(U14G-GPIO_EMC_15-PadB1) -> /EXT_IO16_UART1_RTS
- U14 pad B11: /imxrt10-schematic/UART4_TX -> /USART3_RX
- U14 pad B12: /imxrt10-schematic/SPI4_SCK -> /esp32_wifi_section/IO6_SPI_CLK
- U14 pad B14: unconnected-(U14D-GPIO_B1_15-PadB14) -> /esp32_wifi_section/IO4_DATA_RDY
- U14 pad B2: unconnected-(U14G-GPIO_EMC_18-PadB2) -> /USART3_RTS
- U14 pad B3: unconnected-(U14G-GPIO_EMC_26-PadB3) -> /EXT_IO21
- U14 pad B9: unconnected-(U14D-GPIO_B0_08-PadB9) -> /EXT_IO15_UART1_TX
- U14 pad C12: /imxrt10-schematic/SPI4_SDO -> /esp32_wifi_section/IO7_SPI_MOSI
- U14 pad C4: unconnected-(U14G-GPIO_EMC_33-PadC4) -> /EXT_IO25
- U14 pad C6: unconnected-(U14G-GPIO_EMC_30-PadC6) -> /imxrt10-schematic/SPI1_CS0
- U14 pad C9: unconnected-(U14D-GPIO_B0_09-PadC9) -> /EXT_IO14_UART1_RX
- U14 pad D1: unconnected-(U14G-GPIO_EMC_28-PadD1) -> /imxrt10-schematic/SPI1_SDO
- U14 pad D12: /imxrt10-schematic/SPI4_SDI -> /esp32_wifi_section/IO2_SPI_MISO
- U14 pad D14: unconnected-(U14D-GPIO_B1_13-PadD14) -> /EXT_IO18
- U14 pad D3: unconnected-(U14G-GPIO_EMC_24-PadD3) -> /imxrt10-schematic/UART5_RX
- U14 pad D5: unconnected-(U14G-GPIO_EMC_32-PadD5) -> /EXT_IO22
- U14 pad D6: unconnected-(U14G-GPIO_EMC_38-PadD6) -> /EXT_IO27
- U14 pad D8: unconnected-(U14D-GPIO_B0_03-PadD8) -> /EXT_IO23_CAN_TX
- U14 pad E1: unconnected-(U14G-GPIO_EMC_29-PadE1) -> /imxrt10-schematic/SPI1_SDI
- U14 pad E12: /imxrt10-schematic/SPI4_CS0 -> /esp32_wifi_section/IO10_CS
- U14 pad E3: unconnected-(U14G-GPIO_EMC_00-PadE3) -> /EXT_IO11_SPI_SCK
- U14 pad E8: unconnected-(U14D-GPIO_B0_02-PadE8) -> /EXT_IO24_CAN_RX
- U14 pad F3: unconnected-(U14G-GPIO_EMC_01-PadF3) -> /EXT_IO8_SPI_CS
- U14 pad F4: unconnected-(U14G-GPIO_EMC_02-PadF4) -> /EXT_IO9_SPI_MISO
- U14 pad G12: /esp32_wifi_section/IO7_SPI_MOSI -> /imxrt10-schematic/SPI3_SDO
- U14 pad G2: unconnected-(U14G-GPIO_EMC_23-PadG2) -> /imxrt10-schematic/UART5_TX
- U14 pad G4: unconnected-(U14G-GPIO_EMC_03-PadG4) -> /EXT_IO10_SPI_MOSI
- U14 pad H10: /esp32_wifi_section/IO4_DATA_RDY -> /imxrt10-schematic/SPI3_TRG
- U14 pad H11: /esp32_wifi_section/IO2_SPI_MISO -> /imxrt10-schematic/SPI3_SDI
- U14 pad H12: /esp32_wifi_section/IO10_CS -> /imxrt10-schematic/SPI3_CS0
- U14 pad H13: unconnected-(U14E-GPIO_AD_B1_08-PadH13) -> /EXT_IO6
- U14 pad H4: unconnected-(U14G-GPIO_EMC_07-PadH4) -> /EXT_IO19
- U14 pad J11: /I2C1_SCL -> /EXT_IO0_I2C0_SCL
- U14 pad J12: /imxrt10-schematic/I2C3_SDA -> /EXT_IO2_I2C1_SDA
- U14 pad J13: unconnected-(U14E-GPIO_AD_B1_11-PadJ13) -> /imxrt10-schematic/ADC_IN0
- U14 pad J14: /esp32_wifi_section/IO6_SPI_CLK -> /imxrt10-schematic/SPI3_SCK
- U14 pad K10: /imxrt10-schematic/I2C3_SCL -> /EXT_IO3_I2C1_SCL
- U14 pad K11: /I2C1_SDA -> /EXT_IO1_I2C0_SDA
- U14 pad K12: unconnected-(U14E-GPIO_AD_B1_05-PadK12) -> /EXT_IO5
- U14 pad L11: /imxrt10-schematic/UART2_TX -> /EXT_IO26_UART2_RX
- U14 pad L12: unconnected-(U14E-GPIO_AD_B1_04-PadL12) -> /EXT_IO4
- U14 pad L13: unconnected-(U14E-GPIO_AD_B1_10-PadL13) -> /EXT_IO12
- U14 pad M12: /imxrt10-schematic/UART2_RX -> /EXT_IO13_UART2_TX
- U14 pad M13: unconnected-(U14E-GPIO_AD_B1_09-PadM13) -> /EXT_IO7
- U14 pad M14: unconnected-(U14E-GPIO_AD_B0_00-PadM14) -> /imxrt10-schematic/LED1
- U16 pad 2: TEM_AN0 -> /imxrt10-schematic/ADC_IN0
- U30 pad 1: VDD -> +3.3V1
- U30 pad 10: unconnected-(U30-PA0-Pad10) -> /stm32f103-mcu-interface/NTC_TEMP
- U30 pad 18: unconnected-(U30-PB0-Pad18) -> /stm32f103-mcu-interface/DIN
- U30 pad 2: /stm32f103-mcu-interface/DIN -> /stm32f103-mcu-interface/LED3
- U30 pad 24: VDD -> +3.3V1
- U30 pad 25: /imxrt10-schematic/SPI4_CS0 -> /imxrt10-schematic/SPI1_CS0
- U30 pad 26: /imxrt10-schematic/SPI4_SCK -> /imxrt10-schematic/SPI1_SCK
- U30 pad 27: /imxrt10-schematic/SPI4_SDI -> /imxrt10-schematic/SPI1_SDI
- U30 pad 28: /imxrt10-schematic/SPI4_SDO -> /imxrt10-schematic/SPI1_SDO
- U30 pad 30: /imxrt10-schematic/UART4_RX -> /imxrt10-schematic/UART5_RX
- U30 pad 31: /imxrt10-schematic/UART4_TX -> /imxrt10-schematic/UART5_TX
- U30 pad 36: VDD -> +3.3V1
- U30 pad 48: VDD -> +3.3V1
- U30 pad 9: VDD -> +3.3V1
- U4 pad 3: +3.3V -> +3.3V1
- U5 pad 1: +3.3V -> +3.3V1
- U6 pad 4: unconnected-(U6-XTAL_32K_P-Pad4) -> /esp32_wifi_section/ESP_STATUS_LED
Routing:
- net VBUS: track 4.23 -> 192.1 mm, vias 0 -> 8
- net GND: track 16.4 -> 183.9 mm, vias 20 -> 96
- net /EXT_IO21: track 0.00 -> 88.5 mm, vias 0 -> 2
- net /EXT_IO26_UART2_RX: track 0.00 -> 87.4 mm, vias 0 -> 1
- net /esp32_wifi_section/ESP_TX: track 0.00 -> 83.1 mm, vias 0 -> 5
- net /EXT_IO1_I2C0_SDA: track 0.00 -> 79.0 mm, vias 0 -> 4
- net /esp32_wifi_section/ESP_RX: track 0.00 -> 77.7 mm, vias 0 -> 5
- net /EXT_IO13_UART2_TX: track 0.00 -> 77.1 mm, vias 0 -> 1
- net VBUS_HOST: track 0.00 -> 75.4 mm, vias 0 -> 5
- net /esp32_wifi_section/IO2_SPI_MISO: track 0.00 -> 72.0 mm, vias 0 -> 5
- net /EXT_IO0_I2C0_SCL: track 0.00 -> 71.2 mm, vias 0 -> 4
- net /EXT_IO19: track 0.00 -> 68.1 mm, vias 0 -> 3
- net /esp32_wifi_section/IO4_DATA_RDY: track 0.00 -> 65.2 mm, vias 0 -> 2
- net /imxrt10-schematic/USB_HOST_PWR_OC: track 0.00 -> 65.1 mm, vias 0 -> 4
- net /esp32_wifi_section/IO6_SPI_CLK: track 0.00 -> 64.5 mm, vias 0 -> 2
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- added copper zone on In2.Cu, net GND
Other:
- board size 100 x 59.8 mm -> 100.8 x 75 mm

Commit message: Update the pcb routing
Parts:
- removed JP1, JP2: JUMP, External_Library:power-jumper-3
Connections:
- C32 pad 1: Net-(JP2-B) -> VBUS
- C33 pad 1: /power-supply/+3.3V2 -> +3.3V
- C34 pad 1: Net-(JP2-A) -> VBUS
- C35 pad 1: Net-(JP2-A) -> VBUS
- C37 pad 1: /power-supply/FB -> +3.3V_SYS
- C38 pad 1: /power-supply/FB -> +3.3V_SYS
- C39 pad 1: +3.3V1 -> +3.3V_MPU
- C40 pad 1: +3.3V1 -> +3.3V_MPU
- C43 pad 1: +3.3V1 -> +3.3V_MPU
- L2 pad 2: /power-supply/FB -> +3.3V_SYS
- Q6 pad 1: unconnected-(Q6-G-Pad1) -> /EXT_PWR_EN
- Q8 pad 3: +3.3V1 -> +3.3V_MPU
- R17 pad 1: +3.3V1 -> +3.3V_MPU
- R18 pad 1: +3.3V1 -> +3.3V_MPU
- U10 pad 1: +3.3V1 -> +3.3V_MPU
- U10 pad 6: +3.3V1 -> +3.3V_MPU
- U10 pad 7: +3.3V1 -> +3.3V_MPU
- U14 pad A12: unconnected-(U14D-GPIO_B1_08-PadA12) -> /MPU_INT
- U14 pad D13: unconnected-(U14D-GPIO_B1_12-PadD13) -> /EXT_PWR_EN
- U7 pad 2: /power-supply/+3.3V2 -> +3.3V
- U7 pad 3: Net-(JP2-B) -> VBUS
- U8 pad 1: /power-supply/FB -> +3.3V_SYS
- U8 pad 2: Net-(JP2-A) -> VBUS
- U8 pad 3: Net-(JP2-A) -> VBUS
Routing:
- net +3.3V_SYS: track 12.0 -> 162.8 mm, vias 0 -> 9
- net +3.3V: track 50.1 -> 82.8 mm, vias 11 -> 36
- net GND: track 183.9 -> 216.4 mm, vias 96 -> 111
- net /MPU_INT: track 0.00 -> 25.9 mm, vias 0 -> 2
- net VBUS: track 192.1 -> 217.5 mm, vias 8 -> 9
- net unconnected-(U14D-GPIO_B1_08-PadA12): track 25.0 -> 0.00 mm, vias 2 -> 0
- net /EXT_PWR_EN: track 0.00 -> 21.5 mm, vias 0 -> 2
- net Net-(JP2-A): track 21.0 -> 0.00 mm, vias 6 -> 0
- net /power-supply/FB: track 20.4 -> 0.00 mm, vias 5 -> 0
- net +3.3V_MPU: track 0.00 -> 17.7 mm
- net /power-supply/+3.3V2: track 14.1 -> 0.00 mm, vias 4 -> 0
- net +3.3V1: track 59.6 -> 51.5 mm, vias 0 -> 9
- net Net-(JP2-B): track 5.24 -> 0.00 mm, vias 1 -> 0
- net /esp32_wifi_section/ESP_TX: track 83.1 -> 80.0 mm
- net /esp32_wifi_section/ESP_RX: track 77.7 -> 75.4 mm
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- added copper zone on In2.Cu, net +3.3V
- added copper zone on In2.Cu, net +3.3V1
- added copper zone on F.Cu, net +3.3V_SYS
- added copper zone on B.Cu, net GND
- added copper zone on In1.Cu, net GND
- added copper zone on F.Cu, net VBUS
- removed copper zone on F.Cu, net /power-supply/FB
- removed copper zone on In2.Cu, net GND
- removed copper zone on F.Cu, net Net-(JP2-A)

Commit message: Layout improvement
Connections:
- Q5 pad 1: /modules-sections/WIZ_PWEN -> /WIZ_PWEN
- U30 pad 41: unconnected-(U30-PB5-Pad41) -> /WIZ_PWEN
Routing:
- net /WIZ_PWEN: track 0.00 -> 26.9 mm, vias 0 -> 4
- net VBUS: track 217.5 -> 216.6 mm
- net Net-(U14H-DCDC_IN_Q): track 15.6 -> 14.9 mm
Other:
- board size 100.8 x 75 mm -> 100 x 74 mm
