File: imxrt10-mcu-board-design.kicad_sch (KiCad schematic)
At the start: 14 parts, among them U5 MCP9701T-E/TT

Commit message: Update the source code
Parts:
- added C45, C68, C92, C98: 100n, Capacitor_SMD:C_0603_1608Metric, symbol Device:C_Small
- added D10: LED, Yellow, LED_SMD:LED_0603_1608Metric, symbol Device:LED
- added D8: LED, RED, LED_SMD:LED_0603_1608Metric, symbol Device:LED
- added D9: LED, White, LED_SMD:LED_0603_1608Metric, symbol Device:LED
- added J6: MSD-4-A, External_Library:CUI_MSD-4-A, symbol External_Library:MSD-4-A
- added R1, R2, R33, R34: 10K, Resistor_SMD:R_0603_1608Metric, symbol Device:R
- added R29, R30, R38: 750R, Resistor_SMD:R_0603_1608Metric, symbol Device:R
- added U13: SHT4x, Sensor_Humidity:Sensirion_DFN-4_1.5x1.5mm_P0.8mm_SHT4x_NoCentralPad, symbol Sensor_Humidity:SHT4x
- added U17: W25Q128JVS, Package_SO:SOIC-8_3.9x4.9mm_P1.27mm, symbol Memory_Flash:W25Q128JVS
- added U20: APS1604M-3SQRx-SN, Package_SO:SOIC-8_3.9x4.9mm_P1.27mm, symbol Memory_RAM:APS1604M-3SQRx-SN
Connections:
- net +3.3V: now also C45.1, C68.1, C92.1, C98.1, J6.4 (VDD), R1.1, R2.1, R33.1, R34.1, U13.3 (VDD), U17.8 (VCC), U20.8 (VDD)
- net GND: now also C45.2, C68.2, C92.2, C98.2, D10.1 (K), D8.1 (K), D9.1 (K), J6.6 (VSS), J6.G1 (COVER_GND), J6.G2 (COVER_GND), J6.G3 (COVER_GND), J6.G4 (COVER_GND), U13.4 (VSS), U17.4 (GND), U20.4 (VSS)
- net I2C1_SCL: now also R1.2, U13.2 (SCL)
- net I2C1_SDA: now also R2.2, U13.1 (SDA)
- net LED1: now also R38.2
- net LED2: now also R29.2
- net LED3: now also R30.2
- net SD_CMD: now also J6.3 (CMD)
- net SD_D0: now also J6.7 (DAT0)
- net SD_D1: now also J6.8 (DAT1)
- net SD_D2: now also J6.1 (DAT2)
- net SD_D3: now also J6.2 (CD/DAT3)
- net SD_SCK: now also J6.5 (CLK)
- new net: D8.2 (A), R38.1
- new net: D9.2 (A), R29.1
- new net: D10.2 (A), R30.1
- new net FLEXSPI_A_CLK: U17.6 (CLK)
- new net FLEXSPI_A_SD0: U17.5 (DI(IO0))
- new net FLEXSPI_A_SD1: U17.2 (DO(IO1))
- new net FLEXSPI_A_SD2: U17.3 (IO2)
- new net FLEXSPI_A_SD3: U17.7 (IO3)
- new net FLEXSPI_A_SS: R33.2, U17.1 (~{CS})
- new net FLEXSPI_B_CLK: U20.6 (SCLK)
- new net FLEXSPI_B_SD0: U20.5 (SI/SIO0)
- new net FLEXSPI_B_SD1: U20.2 (SO/SIO1)
- new net FLEXSPI_B_SD2: U20.3 (SIO2)
- new net FLEXSPI_B_SD3: U20.7 (SIO3)
- new net FLEXSPI_B_SS: R34.2, U20.1 (~{CE})
- new net SD_CD: J6.CD
- no-connect marks 5 -> 6
Other:
- sheet esp32_wifi_section ports: added IO10_CS, IO2_SPI_MISO, IO3_HS, IO4_DATA_RDY, IO6_SPI_CLK, IO7_SPI_MOSI, RST; removed none
- sheet imxrt10-schematic ports: added I2C1_SCL, I2C1_SDA, SPI3_CS0, SPI3_SCK, SPI3_SDI, SPI3_SDO, SPI3_TRG, SPI4_CS0, SPI4_SCK, SPI4_SDI, SPI4_SDO, UART4_RX, UART4_TX, UART6_RX, UART6_TX; removed none
- note added: "PSRAM"
- note added: "SD Card"
- note added: "SPI Flash"
- note added: "STM32 MCU"
- moved on the sheet: JP1

Commit message: Update the source code
Parts:
- removed U5: MCP9701T-E/TT, Package_TO_SOT_SMD:SOT-23, symbol Sensor_Temperature:MCP9700AT-ETT
- C68, R1, R2: now fitted
Other:
- added sheet stm32f103-mcu-interface (stm32f103-mcu-interface.kicad_sch)
- sheet modules-sections ports: added WIZ_SPI_CS, WIZ_SPI_INT, WIZ_SPI_MISO, WIZ_SPI_MOSI, WIZ_SPI_SCK; removed LORA_D0, LORA_D1, LORA_D2, LORA_D3, LORA_D4, LORA_D5, LORA_MISO, LORA_MOSI, LORA_NSS, LORA_RST, LORA_SCK, SD_CMD, SD_D0, SD_D1, SD_D2, SD_D3, SD_SCK
- moved on the sheet: C21, D1, R3, TH1

Commit message: Update the schematic
Parts:
- added D13: SS34, PCM_JLCPCB:D_SMA, symbol PCM_JLCPCB-Diodes:Schottky,SS34
- added J1: Conn_02x20_Odd_Even, Connector_PinHeader_2.54mm:PinHeader_2x20_P2.54mm_Vertical, symbol Connector_Generic:Conn_02x20_Odd_Even
- added Q1, Q2: HL3401, PCM_JLCPCB:Q_SOT-23, symbol PCM_JLCPCB-Transistors:PMOS,HL3401
- added R41, R42, R45: 10K, Resistor_SMD:R_0603_1608Metric, symbol Device:R
Connections:
- net +3.3V: no longer C45.1, J6.4 (VDD)
- net GND: now also J1.14 (Pin_14), J1.20 (Pin_20), J1.25 (Pin_25), J1.30 (Pin_30), J1.34 (Pin_34), J1.39 (Pin_39), J1.6 (Pin_6), J1.9 (Pin_9), R41.2, R42.2
- net VBUS: now also D13.2
- new net: D13.1, J1.2 (Pin_2), J1.4 (Pin_4)
- new net +3.3V_EXT: J1.1 (Pin_1), J1.17 (Pin_17), Q2.3 (D)
- new net +3.3V_SD: C45.1, J6.4 (VDD), Q1.3 (D)
- new net +3.3V_SYS: Q1.2 (S), Q2.2 (S), R45.1
- new net EXT_IO0_I2C0_SCL: J1.28 (Pin_28)
- new net EXT_IO10_SPI_MOSI: J1.19 (Pin_19)
- new net EXT_IO11_SPI_SCK: J1.23 (Pin_23)
- new net EXT_IO12: J1.32 (Pin_32)
- new net EXT_IO13_UART2_TX: J1.33 (Pin_33)
- new net EXT_IO14_UART1_RX: J1.8 (Pin_8)
- new net EXT_IO15_UART1_TX: J1.10 (Pin_10)
- new net EXT_IO16_UART1_RTS: J1.36 (Pin_36)
- new net EXT_IO17_UART1_CTS: J1.11 (Pin_11)
- new net EXT_IO18: J1.12 (Pin_12)
- new net EXT_IO19: J1.35 (Pin_35)
- new net EXT_IO1_I2C0_SDA: J1.27 (Pin_27)
- new net EXT_IO20: J1.38 (Pin_38)
- new net EXT_IO21: J1.40 (Pin_40)
- new net EXT_IO22: J1.15 (Pin_15)
- new net EXT_IO23_CAN_TX: J1.16 (Pin_16)
- new net EXT_IO24_CAN_RX: J1.18 (Pin_18)
- new net EXT_IO25: J1.22 (Pin_22)
- new net EXT_IO26_UART2_RX: J1.37 (Pin_37)
- new net EXT_IO27: J1.13 (Pin_13)
- new net EXT_IO2_I2C1_SDA: J1.3 (Pin_3)
- new net EXT_IO3_I2C1_SCL: J1.5 (Pin_5)
- new net EXT_IO4: J1.7 (Pin_7)
- new net EXT_IO5: J1.29 (Pin_29)
- new net EXT_IO6: J1.31 (Pin_31)
- new net EXT_IO7: J1.26 (Pin_26)
- new net EXT_IO8_SPI_CS: J1.24 (Pin_24)
- new net EXT_IO9_SPI_MISO: J1.21 (Pin_21)
- new net SD_EN: Q1.1 (G), Q2.1 (G), R41.1, R42.1, R45.2
- no-connect marks 6 -> 2
Other:
- note added: "External GPIO INTERFACE STM32MP1/2 DK Compatible"
- note added: "I2C TEMP SENSOR"
- note removed: "The diode will prevent reverse current from the board to the connected PC portwhen the power is already powered."
- moved on the sheet: C21, C45, C68, C92, C98, D1, D10, D8, D9, J6, JP1, R1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

Commit message: update the design
Parts:
- removed C21: 100n, Capacitor_SMD:C_0603_1608Metric, symbol Device:C_Small
- removed D1: Inolux_IN-PI554FCH, LED_SMD:LED_Inolux_IN-PI554FCH_PLCC4_5.0x5.0mm_P3.2mm, symbol LED:Inolux_IN-PI554FCH
- removed D10, D4: LED, Yellow, LED_SMD:LED_0603_1608Metric, symbol Device:LED
- removed D2, D8: LED, RED, LED_SMD:LED_0603_1608Metric, symbol Device:LED
- removed D3, D9: LED, White, LED_SMD:LED_0603_1608Metric, symbol Device:LED
- removed R29, R30, R38, R4, R5, R6: 750R, Resistor_SMD:R_0603_1608Metric, symbol Device:R
- removed R3, R42: 10K, Resistor_SMD:R_0603_1608Metric, symbol Device:R
- removed TH1: Thermistor_NTC 10k, Resistor_SMD:R_0805_2012Metric, symbol Device:Thermistor_NTC
- added H1, H2, H3, H4: MountingHole_Pad, MountingHole:MountingHole_2.5mm_Pad, symbol Mechanical:MountingHole_Pad
- added Q4, Q6: 2N7002K, PCM_JLCPCB:Q_SOT-23, symbol PCM_JLCPCB-Transistors:NMOS,2N7002K
- C68: footprint Capacitor_SMD:C_0603_1608Metric -> Capacitor_SMD:C_0402_1005Metric
- R1, R2: footprint Resistor_SMD:R_0603_1608Metric -> Resistor_SMD:R_0402_1005Metric
Connections:
- net I2C1_SCL is gone; now on net EXT_IO0_I2C0_SCL: R1.2, U13.2 (SCL)
- net I2C1_SDA is gone; now on net EXT_IO1_I2C0_SDA: R2.2, U13.1 (SDA)
- net +3.3V_SYS: now also R41.1
- net GND: now also Q4.2 (S), Q6.2 (S); no longer R41.2
- net SD_EN: now also Q4.1 (G); no longer Q1.1 (G), Q2.1 (G), R41.1, R45.2
- new net: Q2.1 (G), Q6.3 (D), R45.2
- new net: Q1.1 (G), Q4.3 (D), R41.2
- no-connect marks 2 -> 10
Other:
- sheet imxrt10-schematic ports: added ADC_IN10, ADC_IN13, ADC_IN14, ADC_IN15, ADC_IN9, CAN_RX, CAN_TX, GPIO_B1_13_06, GPIO_EMC_07, GPIO_EMC_13, GPIO_EMC_26, GPIO_EMC_32, GPIO_EMC_33, GPIO_EMC_38, I2C2_SCL, I2C2_SDA, I2C3_SCL, I2C3_SDA, MPU_INT, SPI1_CS0, SPI1_SCK, SPI1_SDI, SPI1_SDO, SPI2_CS0, SPI2_SCK, SPI2_SDI, SPI2_SDO, SPI4_TRG, UART2_RX, UART2_TX, UART3_CTS, UART3_RTS, UART3_RX, UART3_TX, UART4_CTS, UART4_RTS, UART5_RX, UART5_TX; removed none
- note removed: "Status LED"
- moved on the sheet: R41

Commit message: Update the pcb routing
Parts:
- removed JP1: JUMP, External_Library:power-jumper-3, symbol Jumper:Jumper_3_Open
Connections:
- net EXT_PWR_EN: now reaches Q6.1 (G)
Other:
- sheet imxrt10-schematic ports: added GPIO_B1_12; removed none

Commit message: Layout improvement
Other:
- sheet modules-sections ports: added MPU_PWEN, WIZ_PWEN; removed none
- sheet stm32f103-mcu-interface ports: added BOOT0, PB5_PWR_EN; removed none
Changed lines of the file:
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@@
 	(wire
 		(pts
+			(xy 364.49 361.95) (xy 375.92 361.95)
+		)
+		(stroke
+			(width 0)
+			(type default)
+		)
+	)
+	(wire
+		(pts
 			(xy 347.98 237.49) (xy 365.76 237.49)
 		)
@@
 	(wire
 		(pts
+			(xy 351.79 217.17) (xy 365.76 217.17)
+		)
+		(stroke
+			(width 0)
+			(type default)
+		)
+	)
+	(wire
+		(pts
 			(xy 109.22 63.5) (xy 109.22 66.04)
 		)
@@
 		)
 	)
+	(label "WIZ_PWEN"
+		(at 364.49 361.95 0)
+		(effects
+			(font
+				(size 1.27 1.27)
+			)
+			(justify left bottom)
+		)
+	)
 	(label "EXT_IO1_I2C0_SDA"
 		(at 78.74 170.18 0)
@@
 		)
 	)
+	(label "WIZ_PWEN"
+		(at 351.79 217.17 0)
+		(effects
+			(font
+				(size 1.27 1.27)
+			)
+			(justify left bottom)
+		)
+	)
 	(label "EXT_IO4"
 		(at 58.42 71.12 0)
@@
 			)
 		)
+		(pin "BOOT0" input
+			(at 375.92 344.17 180)
+			(effects
+				(font
+					(size 1.27 1.27)
+				)
+				(justify left)
+			)
+		)
+		(pin "PB5_PWR_EN" input
+			(at 375.92 361.95 180)
+			(effects
+				(font
+					(size 1.27 1.27)
+				)
+				(justify left)
+			)
+		)
 		(instances
 			(project "imxrt10-mcu-board-design"
@@
 			(effects
 				(font
+					(size 1.27 1.27)
+				)
+				(justify left)
+			)
+		)
+		(pin "MPU_PWEN" bidirectional
+			(at 365.76 257.81 180)
+			(effects
+				(font
+					(size 1.27 1.27)
+				)
+				(justify left)
+			)
+		)
+		(pin "WIZ_PWEN" bidirectional
+			(at 365.76 217.17 180)
+			(effects
+				(font
