File: stm32f103-mcu-interface.kicad_sch (KiCad schematic)
At the start: 37 parts, among them U2 SPX3819M5-L-3-3, U3 BOOST-MT3608, U30 STM32F103C8Tx, U4 SHT4x, U5 MCP9701T-E/TT

Commit message: update the design
Parts:
- removed C1: 470n, Capacitor_SMD:C_0603_1608Metric, symbol Device:C
- removed C56: 10uF, Capacitor_SMD:C_0603_1608Metric, symbol Device:C_Small
- removed C58: 2.2u, Capacitor_SMD:C_0402_1005Metric, symbol Device:C_Small
- removed C67: 100n, Capacitor_SMD:C_0603_1608Metric, symbol Device:C_Small
- removed D14: LED, LED_SMD:LED_0603_1608Metric, symbol Device:LED
- removed R11: 0R, Resistor_SMD:R_0603_1608Metric, symbol Device:R
- removed R16: 1k, Resistor_SMD:R_0603_1608Metric, symbol Device:R
- added C1: 100n, Capacitor_SMD:C_0603_1608Metric, symbol Device:C_Small
- added D10: LED, Yellow, LED_SMD:LED_0603_1608Metric, symbol Device:LED
- added J2: Conn_ST_STDC14, Connector_PinHeader_1.27mm:PinHeader_2x07_P1.27mm_Vertical, symbol Connector:Conn_ST_STDC14
- added R27: 750R, Resistor_SMD:R_0603_1608Metric, symbol Device:R
- added R3: 10K, Resistor_SMD:R_0603_1608Metric, symbol Device:R
- added TH1: Thermistor_NTC 10k, Resistor_SMD:R_0805_2012Metric, symbol Device:Thermistor_NTC
Connections:
- net VDD is gone; now on net +3.3V1: C12.1, C14.1, C2.1, C20.1, C3.1, C6.1, C7.1, C8.1, C9.1, D16.1 (VDD), L4.1, R39.1, U2.5 (OUT), U3.5 (IN), U30.1 (VBAT), U30.24 (VDD), U30.36 (VDD), U30.48 (VDD), U30.9 (VDDA)
- net DIN: now also U30.18 (PB0); no longer U30.2 (PC13)
- net GND: now also C1.2, D10.1 (K), J2.11 (GNDDetect), J2.5 (GND), J2.7 (GND), TH1.2
- net NRST: now also J2.12 (~{RST})
- net SWCLK: now also J2.6 (JCLK/SWCLK)
- net SWDIO: now also J2.4 (JTMS/SWDIO)
- net UART2_RX: now also J2.13 (VCP_RX)
- net UART2_TX: now also J2.14 (VCP_TX)
- net NTC_TEMP: now reaches U30.10 (PA0)
- net NTC_TEMP: now also R3.2, TH1.1
- net +3.3V renamed +3.3V1
- net +3.3V1: now also C1.1, J2.3 (VCC), R3.1
- net +VBUSF renamed VBUS
- new net: D10.2 (A), R27.1
- new net LED3: R27.2, U30.2 (PC13)
- no-connect marks 26 -> 28
Other:
- moved on the sheet: C11, R15, R40, U4

Commit message: Layout improvement
Connections:
- net PB5_PWR_EN: now reaches U30.41 (PB5)
- no-connect marks 28 -> 27
Changed lines of the file:
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@@
-	)
-	(no_connect
-		(at 73.66 146.05)
 	)
 	(no_connect
@@
 		(pts
 			(xy 59.69 81.28) (xy 59.69 78.74)
+		)
+		(stroke
+			(width 0)
+			(type default)
+		)
+	)
+	(wire
+		(pts
+			(xy 73.66 146.05) (xy 83.82 146.05)
 		)
 		(stroke
@@
 		(effects
 			(font
+				(size 1.27 1.27)
+			)
+			(justify left)
+		)
+	)
+	(hierarchical_label "PB5_PWR_EN"
+		(shape input)
+		(at 83.82 146.05 0)
+		(effects
+			(font
