File: STM32/BEOU.kicad_sch (KiCad schematic)
At the start: 49 parts, among them J1 UART, J2 UART, J3 SPI, U1 STM32F103C8Tx, U2 SPX3819M5-L-3-3, U3 BOOST-MT3608, U4 Temp Senor LM35-D, X1 8MHz

Commit message: update the design
Parts:
- removed C10, C4: 470n, Capacitor_SMD:C_0603_1608Metric, symbol Device:C
- removed C11, C13, C15, C6, C7, C8: 100n, Capacitor_SMD:C_0603_1608Metric, symbol Device:C
- removed C12, C5: 10u, Capacitor_SMD:C_0805_2012Metric, symbol Device:C
- removed C14, C16, C20: 22u, Capacitor_SMD:C_0603_1608Metric, symbol Device:C
- removed C17, C2: 1u, Capacitor_SMD:C_0603_1608Metric, symbol Device:C
- removed C18, C19: 15p, Capacitor_SMD:C_0603_1608Metric, symbol Device:C
- removed C3: 10n, Capacitor_SMD:C_0603_1608Metric, symbol Device:C
- removed C9: 10u, Capacitor_SMD:C_0603_1608Metric, symbol Device:C
- removed D1: D, Diode_SMD:D_0201_0603Metric, symbol Device:D
- removed D2: LED, LED_SMD:LED_0603_1608Metric, symbol Device:LED
- removed D3: D_Schottky, Diode_SMD:D_0201_0603Metric, symbol Device:D_Schottky
- removed D4: LED WS2812B, LED_SMD:LED_WS2812B_PLCC4_5.0x5.0mm_P3.2mm, symbol LED:WS2812B
- removed J1, J2: UART, Connector_PinHeader_2.54mm:PinHeader_1x04_P2.54mm_Vertical, symbol Connector_Generic:Conn_01x04
- removed J3: SPI, Connector_JST:JST_EH_B6B-EH-A_1x06_P2.50mm_Vertical, symbol Connector_Generic:Conn_01x06
- removed L1: 22u, Inductor_SMD:L_0603_1608Metric, symbol Device:L
- removed R10, R11, R12, R13, R14, R15, R16, R5, R6: 220, Resistor_SMD:R_0201_0603Metric, symbol Device:R
- removed R3: 1k, Resistor_SMD:R_0603_1608Metric, symbol Device:R
- removed R4: 5k, Resistor_SMD:R_0603_1608Metric, symbol Device:R
- removed R7: 1k, Resistor_SMD:R_0201_0603Metric, symbol Device:R
- removed R8: 73k, Resistor_SMD:R_0201_0603Metric, symbol Device:R
- removed R9: 10k, Resistor_SMD:R_0201_0603Metric, symbol Device:R
- removed U1: STM32F103C8Tx, Package_QFP:LQFP-48_7x7mm_P0.5mm, symbol MCU_ST_STM32F1:STM32F103C8Tx
- removed U2: SPX3819M5-L-3-3, Package_TO_SOT_SMD:SOT-23-5, symbol Regulator_Linear:SPX3819M5-L-3-3
- removed U3: BOOST-MT3608, Package_TO_SOT_SMD:SOT-23-6, symbol Regulator_Switching:MT3608
- removed U4: Temp Senor LM35-D, Package_SO:SOIC-8_3.9x4.9mm_P1.27mm, symbol Sensor_Temperature:LM35-D
- removed X1: 8MHz, Crystal:Crystal_SMD_3225-4Pin_3.2x2.5mm, symbol Device:Crystal_GND24
- added Q1: PMOS, symbol Simulation_SPICE:PMOS
- added Q3: NMOS, symbol Simulation_SPICE:NMOS
- added V1: 3.3, symbol Simulation_SPICE:VDC
- added V2: VPULSE, symbol Simulation_SPICE:VPULSE
- C1: value 470n -> 10u; footprint Capacitor_SMD:C_0603_1608Metric -> (none)
- R1: value 0R -> 10k; footprint Resistor_SMD:R_0603_1608Metric -> (none)
- R2: value 100 -> 20; footprint Resistor_SMD:R_0201_0603Metric -> (none)
Connections:
- net GND is gone; now on net 0: C1.2
- net 0: now reaches R2.2
- net 0: now also Q3.3 (S), V1.2, V2.2
- net +VBUS renamed 3.3V
- net 3.3V: now also Q1.3 (S), V1.1; no longer C1.1
- net +VBUSF: no longer names the net of R1.2
- net +VBUSF: now also Q1.2 (G), Q3.1 (D)
- net DIN renamed 3.3V_OPT
- net 3.3V_OPT: now also C1.1, Q1.1 (D)
- new net VDRIVE: Q3.2 (G), V2.1
- no-connect marks 26 -> 0
Other:
- note added: ".ic V(3.3V_OPT)=0.5"
- note removed: "+3V3 LDO REGULATOR"
- note removed: "+3V3 TO +5V BOOST REGULATOR"
- note removed: "CONNECTORS TO LCD, UART, SW, RESET"
- note removed: "CRYSTAL CLK"
- note removed: "DIGITAL LED"
- note removed: "MCU STM32F103C8T6"
- note removed: "THERMAL SENSOR"
